Commit message: fixed bugs related to urdf and launch for arm version of robot

File: segbot_arm_launch/robots/segbot_v2.arm.urdf.xacro (robot description, xacro)
@@ -9,5 +9,4 @@
   <xacro:include filename="$(find segbot_description)/urdf/mounts/hokuyo_mount.urdf.xacro" />
   <xacro:include filename="$(find segbot_description)/urdf/mounts/kinect_mount.urdf.xacro" />
-  <xacro:include filename="$(find segbot_description)/urdf/mounts/sensor_plate_mount.urdf.xacro" />
   <xacro:include filename="$(find jaco_model)/urdf/mico_arm.xacro" />
   <!-- Add the segbot base -->
@@ -24,8 +23,12 @@
     <origin xyz="${1*INCH_TO_M} ${0.5*INCH_TO_M} ${4.5*INCH_TO_M}" rpy="${M_PI/2} ${M_PI/2} 0" />
   </xacro:beam_8020>
-  <!-- Add the hokuyo mount without the beam -->
+  <!-- Add the hokuyo mount without the beam
   <xacro:hokuyo_mount_without_beam name="nav_hokuyo" parent="hokuyo_sonar_sensor_beam" ros_topic="scan" update_rate="10" min_angle="${-(5 * M_PI)/12}" max_angle="${(5 * M_PI)/12}" range="20.0">
     <origin xyz="${0.5*INCH_TO_M} 0 ${SENSOR_BEAM_LENGTH/2*INCH_TO_M}" rpy="${M_PI/2} 0 ${M_PI/2}" />
-  </xacro:hokuyo_mount_without_beam>
+  </xacro:hokuyo_mount_without_beam> -->
+   <!-- Add the hokuyo -->
+  <xacro:hokuyo_mount name="nav_hokuyo" parent="front_left_vertical_beam" length="${SENSOR_BEAM_LENGTH*INCH_TO_M}" ros_topic="scan" update_rate="10" min_angle="${-(5 * M_PI)/12}" max_angle="${(5 * M_PI)/12}">
+    <origin xyz="${1*INCH_TO_M} ${0.5*INCH_TO_M} ${4.5*INCH_TO_M}" rpy="${M_PI/2} ${M_PI/2} 0" />
+  </xacro:hokuyo_mount>
   <!-- Add the sensor plate mount -->
   <xacro:sensor_plate_mount_without_beam parent="hokuyo_sonar_sensor_beam" length="${SENSOR_BEAM_LENGTH*INCH_TO_M}"/>

Commit message: updated segbot_v2 arm to use new hokuyo/sensor plate xacro macros.

File: segbot_arm_launch/robots/segbot_v2.arm.urdf.xacro (robot description, xacro)
@@ -23,12 +23,8 @@
     <origin xyz="${1*INCH_TO_M} ${0.5*INCH_TO_M} ${4.5*INCH_TO_M}" rpy="${M_PI/2} ${M_PI/2} 0" />
   </xacro:beam_8020>
-  <!-- Add the hokuyo mount without the beam
+  <!-- Add the hokuyo mount without the beam -->
   <xacro:hokuyo_mount_without_beam name="nav_hokuyo" parent="hokuyo_sonar_sensor_beam" ros_topic="scan" update_rate="10" min_angle="${-(5 * M_PI)/12}" max_angle="${(5 * M_PI)/12}" range="20.0">
     <origin xyz="${0.5*INCH_TO_M} 0 ${SENSOR_BEAM_LENGTH/2*INCH_TO_M}" rpy="${M_PI/2} 0 ${M_PI/2}" />
-  </xacro:hokuyo_mount_without_beam> -->
-   <!-- Add the hokuyo -->
-  <xacro:hokuyo_mount name="nav_hokuyo" parent="front_left_vertical_beam" length="${SENSOR_BEAM_LENGTH*INCH_TO_M}" ros_topic="scan" update_rate="10" min_angle="${-(5 * M_PI)/12}" max_angle="${(5 * M_PI)/12}">
-    <origin xyz="${1*INCH_TO_M} ${0.5*INCH_TO_M} ${4.5*INCH_TO_M}" rpy="${M_PI/2} ${M_PI/2} 0" />
-  </xacro:hokuyo_mount>
+  </xacro:hokuyo_mount_without_beam>
   <!-- Add the sensor plate mount -->
   <xacro:sensor_plate_mount_without_beam parent="hokuyo_sonar_sensor_beam" length="${SENSOR_BEAM_LENGTH*INCH_TO_M}"/>

Commit message: moved the xtion camera to where it is supposed to be

File: segbot_arm_launch/robots/segbot_v2.arm.urdf.xacro (robot description, xacro)
@@ -71,6 +71,6 @@
   <xacro:kinect_camera name="xtion_camera" parent="arm">
      <!-- <origin xyz="0.05 +0.245 0.75" rpy="0 0.74 ${M_PI/2}" /> -->
-      <origin xyz="-0.245 +0.05 0.75" rpy="0 0.74 0" />
-    </xacro:kinect_camera>
+      <origin xyz="-0.245 +0.165 0.75" rpy="0 0.74 0" />
+  </xacro:kinect_camera>
   <xacro:gazebo_segbot_ros_controllers />
 </robot>

File: segbot_arm_launch/robots/segbot_v2.arm.xacroout.urdf (robot description, URDF)
Before this commit: robot segbot, 59 links, 58 joints
Links:
- removed link laser_obstacle
- link back_base_beam_link: geometry collision box size=0.0254 0.0254 0.3048; visual box size=0.0254 0.0254 0.3048
- link back_left_vertical_beam_link: geometry collision box size=0.0254 0.0254 0.4572; visual box size=0.0254 0.0254 0.4572
- link back_right_vertical_beam_link: geometry collision box size=0.0254 0.0254 0.4572; visual box size=0.0254 0.0254 0.4572
- link base_caster_support_link: geometry collision mesh filename=package://segbot_description/meshes/rmp50-castor-link.dae scale=0.0254 0.0254 0.0254; visual mesh filename=package://segbot_description/meshes/rmp50-castor-link.dae scale=0.0254 0.0254 0.0254
- link base_link: geometry collision mesh filename=package://segbot_description/meshes/rmp50-base-link.dae scale=0.0254 0.0254 0.0254; visual mesh filename=package://segbot_description/meshes/rmp50-base-link.dae scale=0.0254 0.0254 0.0254
- link base_link_left_wheel_link: geometry collision mesh filename=package://segbot_description/meshes/rmp50-left-wheel.dae scale=0.0254 0.0254 0.0254; visual mesh filename=package://segbot_description/meshes/rmp50-left-wheel.dae scale=0.0254 0.0254 0.0254
- link base_link_right_wheel_link: geometry collision mesh filename=package://segbot_description/meshes/rmp50-right-wheel.dae scale=0.0254 0.0254 0.0254; visual mesh filename=package://segbot_description/meshes/rmp50-right-wheel.dae scale=0.0254 0.0254 0.0254
- link battery_box_link: geometry collision box size=0.1778 0.3556 0.2794; visual box size=0.1778 0.3556 0.2794
- link caster_wheel_link: geometry collision mesh filename=package://segbot_description/meshes/rmp50-castor-wheel.dae scale=0.0254 0.0254 0.0254; visual mesh filename=package://segbot_description/meshes/rmp50-castor-wheel.dae scale=0.0254 0.0254 0.0254
- link chassis_base_plate_link: geometry collision box size=0.4064 0.3556 0.00635; visual box size=0.4064 0.3556 0.00635
- link chassis_left_plate_link: geometry collision box size=0.4064 0.1016 0.00635; visual box size=0.4064 0.1016 0.00635
- link chassis_right_plate_link: geometry collision box size=0.4064 0.1016 0.00635; visual box size=0.4064 0.1016 0.00635
- link front_base_beam_link: geometry collision box size=0.0254 0.0254 0.3048; visual box size=0.0254 0.0254 0.3048
- link front_left_vertical_beam_link: geometry collision box size=0.0254 0.0254 0.4572; visual box size=0.0254 0.0254 0.4572
- link front_right_vertical_beam_link: geometry collision box size=0.0254 0.0254 0.4572; visual box size=0.0254 0.0254 0.4572
- link hokuyo_sonar_sensor_beam_link: geometry collision box size=0.0254 0.0254 0.3048; visual box size=0.0254 0.0254 0.3048
- link laptop_base_plate_link: geometry collision box size=0.4064 0.4572 0.003175; visual box size=0.4064 0.4572 0.003175
- link laptop_link: geometry collision box size=0.3048 0.3556 0.01905; visual box size=0.2286 0.3048 0.01905
- link laptop_screen_link: geometry collision box size=0.3048 0.3556 0.01905; visual box size=0.3048 0.2286 0.01905
- link left_laptop_support_beam_link: geometry collision box size=0.0254 0.0254 0.3048; visual box size=0.0254 0.0254 0.3048
- link left_sensor_beam_link: geometry collision box size=0.0254 0.0254 0.762; visual box size=0.0254 0.0254 0.762
- link nav_hokuyo_plate_link: geometry collision box size=0.06 0.12 0.003175; visual box size=0.06 0.12 0.003175
- link nav_hokuyo_sensor_beam_link: geometry collision box size=0.0254 0.0254 0.3048; visual box size=0.0254 0.0254 0.3048
- link nav_kinect_base_plate_link: geometry collision box size=0.1016 0.2286 0.0015875; visual box size=0.1016 0.2286 0.0015875
- link nav_kinect_sensor_beam_link: geometry collision box size=0.0254 0.0254 0.3048; visual box size=0.0254 0.0254 0.3048
- link nav_kinect_standoff_1_link: geometry collision cylinder length=0.0508 radius=0.003175; visual cylinder length=0.0508 radius=0.003175
- link nav_kinect_standoff_2_link: geometry collision cylinder length=0.0508 radius=0.003175; visual cylinder length=0.0508 radius=0.003175
- link nav_kinect_standoff_3_link: geometry collision cylinder length=0.0508 radius=0.003175; visual cylinder length=0.0508 radius=0.003175
- link nav_kinect_standoff_4_link: geometry collision cylinder length=0.0508 radius=0.003175; visual cylinder length=0.0508 radius=0.003175
- link nav_kinect_top_plate_link: geometry collision box size=0.1016 0.2286 0.0015875; visual box size=0.1016 0.2286 0.0015875
- link right_laptop_support_beam_link: geometry collision box size=0.0254 0.0254 0.3048; visual box size=0.0254 0.0254 0.3048
- link right_sensor_beam_link: geometry collision box size=0.0254 0.0254 0.762; visual box size=0.0254 0.0254 0.762
- link top_sensor_beam_link: geometry collision box size=0.0254 0.0254 0.4572; visual box size=0.0254 0.0254 0.4572
Joints:
- removed joint laser_obstacle_joint
- joint xtion_camera_joint: origin xyz=-0.245 +0.05 0.75 rpy=0 0.74 0 -> xyz=-0.245 +0.165 0.75 rpy=0 0.74 0

Commit message: small changes to make it work with latest segbot branch

File: segbot_arm_launch/robots/segbot_v2.arm.urdf.xacro (robot description, xacro)
@@ -67,5 +67,5 @@
   <xacro:kinect_camera name="xtion_camera" parent="arm">
      <!-- <origin xyz="0.05 +0.245 0.75" rpy="0 0.74 ${M_PI/2}" /> -->
-      <origin xyz="-0.245 +0.05 0.75" rpy="0 0.74 0" />
+      <origin xyz="-0.245 +0.165 0.75" rpy="0 0.74 0" />
     </xacro:kinect_camera>
   <xacro:gazebo_segbot_ros_controllers />

File: segbot_arm_launch/robots/segbot_v2.arm.xacroout.urdf (robot description, URDF)
Before this commit: robot segbot, 59 links, 58 joints
Links:
- removed link laser_obstacle
- removed link nav_hokuyo_sensor_beam_link
- link back_base_beam_link: geometry collision box size=0.0254 0.0254 0.3048; visual box size=0.0254 0.0254 0.3048
- link back_left_vertical_beam_link: geometry collision box size=0.0254 0.0254 0.4572; visual box size=0.0254 0.0254 0.4572
- link back_right_vertical_beam_link: geometry collision box size=0.0254 0.0254 0.4572; visual box size=0.0254 0.0254 0.4572
- link base_caster_support_link: geometry collision mesh filename=package://segbot_description/meshes/rmp50-castor-link.dae scale=0.0254 0.0254 0.0254; visual mesh filename=package://segbot_description/meshes/rmp50-castor-link.dae scale=0.0254 0.0254 0.0254
- link base_link: geometry collision mesh filename=package://segbot_description/meshes/rmp50-base-link.dae scale=0.0254 0.0254 0.0254; visual mesh filename=package://segbot_description/meshes/rmp50-base-link.dae scale=0.0254 0.0254 0.0254
- link base_link_left_wheel_link: geometry collision mesh filename=package://segbot_description/meshes/rmp50-left-wheel.dae scale=0.0254 0.0254 0.0254; visual mesh filename=package://segbot_description/meshes/rmp50-left-wheel.dae scale=0.0254 0.0254 0.0254
- link base_link_right_wheel_link: geometry collision mesh filename=package://segbot_description/meshes/rmp50-right-wheel.dae scale=0.0254 0.0254 0.0254; visual mesh filename=package://segbot_description/meshes/rmp50-right-wheel.dae scale=0.0254 0.0254 0.0254
- link battery_box_link: geometry collision box size=0.1778 0.3556 0.2794; visual box size=0.1778 0.3556 0.2794
- link caster_wheel_link: geometry collision mesh filename=package://segbot_description/meshes/rmp50-castor-wheel.dae scale=0.0254 0.0254 0.0254; visual mesh filename=package://segbot_description/meshes/rmp50-castor-wheel.dae scale=0.0254 0.0254 0.0254
- link chassis_base_plate_link: geometry collision box size=0.4064 0.3556 0.00635; visual box size=0.4064 0.3556 0.00635
- link chassis_left_plate_link: geometry collision box size=0.4064 0.1016 0.00635; visual box size=0.4064 0.1016 0.00635
- link chassis_right_plate_link: geometry collision box size=0.4064 0.1016 0.00635; visual box size=0.4064 0.1016 0.00635
- link front_base_beam_link: geometry collision box size=0.0254 0.0254 0.3048; visual box size=0.0254 0.0254 0.3048
- link front_left_vertical_beam_link: geometry collision box size=0.0254 0.0254 0.4572; visual box size=0.0254 0.0254 0.4572
- link front_right_vertical_beam_link: geometry collision box size=0.0254 0.0254 0.4572; visual box size=0.0254 0.0254 0.4572
- link hokuyo_sonar_sensor_beam_link: geometry collision box size=0.0254 0.0254 0.3048; visual box size=0.0254 0.0254 0.3048
- link laptop_base_plate_link: geometry collision box size=0.4064 0.4572 0.003175; visual box size=0.4064 0.4572 0.003175
- link laptop_link: geometry collision box size=0.3048 0.3556 0.01905; visual box size=0.2286 0.3048 0.01905
- link laptop_screen_link: geometry collision box size=0.3048 0.3556 0.01905; visual box size=0.3048 0.2286 0.01905
- link left_laptop_support_beam_link: geometry collision box size=0.0254 0.0254 0.3048; visual box size=0.0254 0.0254 0.3048
- link left_sensor_beam_link: geometry collision box size=0.0254 0.0254 0.762; visual box size=0.0254 0.0254 0.762
- link nav_hokuyo_plate_link: geometry collision box size=0.06 0.12 0.003175; visual box size=0.06 0.12 0.003175
- link nav_kinect_base_plate_link: geometry collision box size=0.1016 0.2286 0.0015875; visual box size=0.1016 0.2286 0.0015875
- link nav_kinect_sensor_beam_link: geometry collision box size=0.0254 0.0254 0.3048; visual box size=0.0254 0.0254 0.3048
- link nav_kinect_standoff_1_link: geometry collision cylinder length=0.0508 radius=0.003175; visual cylinder length=0.0508 radius=0.003175
- link nav_kinect_standoff_2_link: geometry collision cylinder length=0.0508 radius=0.003175; visual cylinder length=0.0508 radius=0.003175
- link nav_kinect_standoff_3_link: geometry collision cylinder length=0.0508 radius=0.003175; visual cylinder length=0.0508 radius=0.003175
- link nav_kinect_standoff_4_link: geometry collision cylinder length=0.0508 radius=0.003175; visual cylinder length=0.0508 radius=0.003175
- link nav_kinect_top_plate_link: geometry collision box size=0.1016 0.2286 0.0015875; visual box size=0.1016 0.2286 0.0015875
- link right_laptop_support_beam_link: geometry collision box size=0.0254 0.0254 0.3048; visual box size=0.0254 0.0254 0.3048
- link right_sensor_beam_link: geometry collision box size=0.0254 0.0254 0.762; visual box size=0.0254 0.0254 0.762
- link top_sensor_beam_link: geometry collision box size=0.0254 0.0254 0.4572; visual box size=0.0254 0.0254 0.4572
Joints:
- removed joint laser_obstacle_joint
- removed joint nav_hokuyo_sensor_beam_joint
- joint nav_hokuyo_plate_joint: parent nav_hokuyo_sensor_beam_link -> hokuyo_sonar_sensor_beam_link
- joint xtion_camera_joint: origin xyz=-0.245 +0.05 0.75 rpy=0 0.74 0 -> xyz=-0.245 +0.165 0.75 rpy=0 0.74 0
