Commit message: Make launchfiles use new MoveIt config
Use some new arguments we added to control what the Kinova launch files bring up
Launch Kinova trajectory controllers instead of our hacked together ones

File: segbot_arm_launch/robots/segbot_v2.arm.urdf (robot description, URDF)
Before this commit: robot segbot, 57 links, 56 joints
Links:
- removed link mico_api_origin
- removed link mico_end_effector
- removed link mico_link_1
- removed link mico_link_2
- removed link mico_link_3
- removed link mico_link_4
- removed link mico_link_5
- removed link mico_link_base
- removed link mico_link_finger_1
- removed link mico_link_finger_2
- removed link mico_link_hand
- added link m1n6s200_end_effector; collision box size=0 0 0; visual box size=0 0 0
- added link m1n6s200_link_1, mass 0.7477; collision mesh filename=package://kinova_description/meshes/shoulder.dae; visual mesh filename=package://kinova_description/meshes/ring_big.STL
- added link m1n6s200_link_2, mass 0.85968; collision mesh filename=package://kinova_description/meshes/arm_mico.dae; visual mesh filename=package://kinova_description/meshes/arm_mico.dae
- added link m1n6s200_link_3, mass 0.606; collision mesh filename=package://kinova_description/meshes/forearm_mico.dae; visual mesh filename=package://kinova_description/meshes/forearm_mico.dae
- added link m1n6s200_link_4, mass 0.1785; collision mesh filename=package://kinova_description/meshes/wrist.dae; visual mesh filename=package://kinova_description/meshes/ring_small.STL
- added link m1n6s200_link_5, mass 0.1785; collision mesh filename=package://kinova_description/meshes/wrist.dae; visual mesh filename=package://kinova_description/meshes/ring_small.STL
- added link m1n6s200_link_6, mass 0.78; collision mesh filename=package://kinova_description/meshes/hand_2finger.dae; visual mesh filename=package://kinova_description/meshes/hand_2finger.dae
- added link m1n6s200_link_base, mass 0.46784; collision mesh filename=package://kinova_description/meshes/base.dae; visual mesh filename=package://kinova_description/meshes/base.dae
- added link m1n6s200_link_finger_1, mass 0.01; collision mesh filename=package://kinova_description/meshes/finger_proximal.dae; visual mesh filename=package://kinova_description/meshes/finger_proximal.dae
- added link m1n6s200_link_finger_2, mass 0.01; collision mesh filename=package://kinova_description/meshes/finger_proximal.dae; visual mesh filename=package://kinova_description/meshes/finger_proximal.dae
- added link m1n6s200_link_finger_tip_1, mass 0.01; collision mesh filename=package://kinova_description/meshes/finger_distal.dae; visual mesh filename=package://kinova_description/meshes/finger_distal.dae
- added link m1n6s200_link_finger_tip_2, mass 0.01; collision mesh filename=package://kinova_description/meshes/finger_distal.dae; visual mesh filename=package://kinova_description/meshes/finger_distal.dae
Joints:
- removed joint mico_joint_1
- removed joint mico_joint_2
- removed joint mico_joint_3
- removed joint mico_joint_4
- removed joint mico_joint_5
- removed joint mico_joint_6
- removed joint mico_joint_base
- removed joint mico_joint_finger_1
- removed joint mico_joint_finger_2
- removed joint mico_link_base_to_api_origin
- removed joint mico_link_hand_to_end_effector
- added joint m1n6s200_joint_1: type continuous, parent m1n6s200_link_base, child m1n6s200_link_1, origin xyz=0 0 0.15675 rpy=0 3.14159265359 0, axis 0 0 1, limit lower=-6.28318530718 upper=6.28318530718 effort=2000 velocity=1
- added joint m1n6s200_joint_2: type revolute, parent m1n6s200_link_1, child m1n6s200_link_2, origin xyz=0 0.0016 -0.11875 rpy=-1.57079632679 0 3.14159265359, axis 0 0 1, limit lower=0.523598775598 upper=5.75958653158 effort=2000 velocity=1
- added joint m1n6s200_joint_3: type revolute, parent m1n6s200_link_2, child m1n6s200_link_3, origin xyz=0 -0.290 0 rpy=0 3.14159265359 0, axis 0 0 1, limit lower=0.523598775598 upper=5.75958653158 effort=2000 velocity=1
- added joint m1n6s200_joint_4: type continuous, parent m1n6s200_link_3, child m1n6s200_link_4, origin xyz=0 0.1231 -0.0086 rpy=-1.57079632679 0 3.14159265359, axis 0 0 1, limit lower=-6.28318530718 upper=6.28318530718 effort=2000 velocity=1
- added joint m1n6s200_joint_5: type continuous, parent m1n6s200_link_4, child m1n6s200_link_5, origin xyz=0 -0.03703 -0.06414 rpy=1.0471975512 0 3.14159265359, axis 0 0 1, limit lower=-6.28318530718 upper=6.28318530718 effort=2000 velocity=1
- added joint m1n6s200_joint_6: type continuous, parent m1n6s200_link_5, child m1n6s200_link_6, origin xyz=0 -0.03703 -0.06414 rpy=1.0471975512 0 3.14159265359, axis 0 0 1, limit lower=-6.28318530718 upper=6.28318530718 effort=2000 velocity=1
- added joint m1n6s200_joint_base: type fixed, parent arm_link, child m1n6s200_link_base, origin xyz=0 0 0 rpy=0 0 0, axis 0 0 0, limit lower=0 upper=0 effort=2000 velocity=1
- added joint m1n6s200_joint_end_effector: type fixed, parent m1n6s200_link_6, child m1n6s200_end_effector, origin xyz=0 0 -0.1600 rpy=3.14159265359 0 0, axis 0 0 0, limit lower=0 upper=0 effort=2000 velocity=1
- added joint m1n6s200_joint_finger_1: type revolute, parent m1n6s200_link_6, child m1n6s200_link_finger_1, origin xyz=-0.0025 0.03095 -0.11482 rpy=-1.570796327 .649262481663582 1.57079632679490, axis 0 0 1, limit lower=0 upper=2 effort=2000 velocity=1
- added joint m1n6s200_joint_finger_2: type revolute, parent m1n6s200_link_6, child m1n6s200_link_finger_2, origin xyz=-0.0025 -0.03095 -0.11482 rpy=-1.570796327 .649262481663582 -1.57079632679490, axis 0 0 1, limit lower=0 upper=2 effort=2000 velocity=1
- added joint m1n6s200_joint_finger_tip_1: type fixed, parent m1n6s200_link_finger_1, child m1n6s200_link_finger_tip_1, origin xyz=0.044 -0.003 0 rpy=0 0 0, axis 0 0 1, limit lower=0 upper=2 effort=2000 velocity=1
- added joint m1n6s200_joint_finger_tip_2: type fixed, parent m1n6s200_link_finger_2, child m1n6s200_link_finger_tip_2, origin xyz=0.044 -0.003 0 rpy=0 0 0, axis 0 0 1, limit lower=0 upper=2 effort=2000 velocity=1

File: segbot_arm_launch/robots/segbot_v2.arm.urdf.xacro (robot description, xacro)
@@ -66,5 +66,5 @@
        the joint names on the /out/joint_states topic
 	-->
-  <xacro:m1n6s200 base_parent="arm_link" prefix="mico"/>
+  <xacro:m1n6s200 base_parent="arm_link"/>
   <!-- add the xtion -->
   <xacro:kinect_camera name="xtion_camera" parent="arm">
