Commit message: added standalone launch for urdf viewing. Vastly improved primitive urdf through bug fixes and more joints to describe the full chain of motors.

File: dynamixel_arm/urdf/dynamixel_arm_primative.urdf (robot description, URDF)
Before this commit: robot dynamixel_arm, 3 links, 2 joints
Links:
- removed link link1_spindle
- added link bottom_mount_1; visual box size=.032 .032 .002
- added link link_1_spindle; visual cylinder length=.04 radius=.004
- added link link_2; visual cylinder length=.005 radius=.0115
- added link link_2_spindle; visual cylinder length=.04 radius=.004
- added link servo_body_2; visual box size=.032 .032 .050
- added link top_mount_1; visual box size=.048 .029 .063
- added link top_mount_2; visual box size=.048 .029 .037
- link base_link: geometry visual box size=.032 .032 .050
- link link_1: geometry visual cylinder length=.005 radius=.0115
Joints:
- removed joint spindle_to_joint1
- added joint body_2_to_spindle: type fixed, parent servo_body_2, child link_2_spindle, origin xyz=0 0 -0.016 rpy=-1.57075 0 0
- added joint bottom_mount_1_to_servo_body_2: type fixed, parent bottom_mount_1, child servo_body_2, origin xyz=0 0.025 0 rpy=1.57075 0 0
- added joint joint_1_to_mount_1: type fixed, parent link_1, child top_mount_1, origin xyz=0 0.020 -0.019
- added joint joint_2_to_mount_2: type fixed, parent link_2, child top_mount_2, origin xyz=0 0.007 -0.019
- added joint mount_1_to_bottom_mount_1: type fixed, parent top_mount_1, child bottom_mount_1, origin xyz=0 .0325 0
- added joint spindle_to_joint_1: type revolute, parent link_1_spindle, child link_1, origin xyz=0 0 0.019, axis 0 0 1, limit lower=-1.57 upper=1.57 effort=1000.0 velocity=1.00
- added joint spindle_to_joint_2: type revolute, parent link_2_spindle, child link_2, origin xyz=0 0 0.019, axis 0 0 1, limit lower=-1.57 upper=1.57 effort=1000.0 velocity=1.00
- joint base_to_spindle: child link1_spindle -> link_1_spindle
