Commit message: package restructuring, including splitting the urdf description into its own package. added additional controller (torque)

File: dynamixel/dynamixel_description/urdf/dynamixel_arm.urdf (robot description, URDF)
Before this commit: robot dynamixel_arm, 2 links, 1 joints
Links:
- link base_link: geometry visual mesh filename=package://dynamixel_description/mesh/ax12_box.dae
- link wheel: geometry visual mesh filename=package://dynamixel_description/mesh/ax12_wheel.dae
